File: PCB/Board Schematics/Kicad schematics (recommended)/OF1 v1.kicad_sch (KiCad schematic)
At the start: 51 parts, among them J1 RPI_PICO-TH, J2 MOLEX2171830001, J3 MA06-1, J4 MA04-1, J5 GT-USB-7010

Commit message: WIP
Parts:
- removed J4: MA04-1, OF1 v1:MA04-1, symbol OF1 v1-eagle-import:MA04-1
- added J4: GT-USB-7010, OF1 v1:16P, symbol OF1 v1-eagle-import:GT-USB-7010ASV
Connections:
- net +5V: no longer J5.A4/B9 (VBUS), J5.B4/A9 (VBUS)
- net D+: no longer J5.A6 (D+), J5.B6 (D+)
- net D-: no longer J5.A7 (D-), J5.B7 (D-)
- net DOWN: now also J4.A8 (SBU1), J4.B8 (SBU2); no longer JP4.1, U$4.P$2 (PIN1), U$4.P$3 (PIN1)
- net GND: now also J4.SHIELD1 (SHIELD), J4.SHIELD2 (SHIELD), J4.SHIELD3 (SHIELD), J4.SHIELD4 (SHIELD); no longer J5.A1/B12 (GND), J5.B1/A12 (GND)
- net L: now also J4.A5 (CC1), J4.B5 (CC2); no longer JP2.1, U$1.P$2 (PIN1), U$1.P$3 (PIN1)
- net LEFT: now also J4.A6 (D+), J4.B6 (D+); no longer JP3.1, U$2.P$2 (PIN1), U$2.P$3 (PIN1)
- net M1: now also J4.A1/B12 (GND), J4.B1/A12 (GND); no longer JP6.1, U$6.P$2 (PIN1), U$6.P$3 (PIN1)
- net M2: now also J4.A4/B9 (VBUS), J4.B4/A9 (VBUS); no longer JP7.1, U$7.P$2 (PIN1), U$7.P$3 (PIN1)
- net RIGHT: now also J4.A7 (D-), J4.B7 (D-); no longer JP5.1, U$5.P$2 (PIN1), U$5.P$3 (PIN1)
- net L_J: now reaches J5.A5 (CC1)
- net L_J: now also J5.B5 (CC2), JP2.1, U$1.P$2 (PIN1), U$1.P$3 (PIN1)
- net RIGHT_J: now reaches J5.A8 (SBU1)
- net RIGHT_J: now also J5.B8 (SBU2), JP5.1, U$5.P$2 (PIN1), U$5.P$3 (PIN1)
- new net DOWN_J: J5.A7 (D-), J5.B7 (D-), JP4.1, U$4.P$2 (PIN1), U$4.P$3 (PIN1)
- new net LEFT_J: J5.A6 (D+), J5.B6 (D+), JP3.1, U$2.P$2 (PIN1), U$2.P$3 (PIN1)
- new net M1_J: J5.A1/B12 (GND), J5.B1/A12 (GND), JP6.1, U$6.P$2 (PIN1), U$6.P$3 (PIN1)
- new net M2_J: J5.A4/B9 (VBUS), J5.B4/A9 (VBUS), JP7.1, U$7.P$2 (PIN1), U$7.P$3 (PIN1)
Other:
- note added: "J6"
